Commit message: map server added

File: src/robot_description/urdf/ubot.xacro (robot description, xacro)
@@ -1,3 +1,158 @@
-<?xml version="1.0" ?>
-<robot name="ubot" xmlns:xacro="http://www.ros.org/wiki/xacro">
+<?xml version="1.0"?>
+<robot xmlns:xacro="http://www.ros.org/wiki/xacro" name="ubot">
+  <xacro:property name="base_width" value="0.16"/>
+  <xacro:property name="base_len" value="0.16"/>
+  <xacro:property name="wheel_radius" value="0.035"/>
+  <xacro:property name="base_wheel_gap" value="0.007"/>
+  <xacro:property name="wheel_separation" value="0.15"/>
+  <xacro:property name="wheel_joint_offset" value="0.02"/>
+  <xacro:property name="caster_wheel_radius" value="${wheel_radius/2}"/>
+  <xacro:property name="caster_wheel_mass" value="0.001"/>
+  <xacro:property name="caster_wheel_joint_offset" value="-0.052"/>
+  <!--Color Properties-->
+  <material name="blue">
+    <color rgba="0 0 0.8 1"/>
+  </material>
+  <material name="black">
+    <color rgba="0 0 0 1"/>
+  </material>
+  <material name="white">
+    <color rgba="1 1 1 1"/>
+  </material>
+  <material name="red">
+    <color rgba="0.8 0.0 0.0 1.0"/>
+  </material>
+  <!--Interial macros-->
+  <xacro:macro name="cylinder_inertia" params="m r h">
+    <inertial>
+      <mass value="${m}"/>
+      <inertia ixx="${m*(3*r*r+h*h)/12}" ixy = "0" ixz = "0" iyy="${m*(3*r*r+h*h)/12}" iyz = "0" izz="${m*r*r/2}"/>
+    </inertial>
+  </xacro:macro>
+  <xacro:macro name="box_inertia" params="m w h d">
+    <inertial>
+      <mass value="${m}"/>
+      <inertia ixx="${m / 12.0 * (d*d + h*h)}" ixy="0.0" ixz="0.0" iyy="${m / 12.0 * (w*w + h*h)}" iyz="0.0" izz="${m / 12.0 * (w*w + d*d)}"/>
+    </inertial>
+  </xacro:macro>
+  <xacro:macro name="sphere_inertia" params="m r">
+    <inertial>
+      <mass value="${m}"/>
+      <inertia ixx="${2.0*m*(r*r)/5.0}" ixy="0.0" ixz="0.0" iyy="${2.0*m*(r*r)/5.0}" iyz="0.0" izz="${2.0*m*(r*r)/5.0}"/>
+    </inertial>
+  </xacro:macro>
+  <!--Base Footprint-->
+  <link name="base_footprint">
+    <xacro:box_inertia m="10" w="0.001" h="0.001" d="0.001"/>
+    <visual>
+        <origin xyz="0 0 0" rpy="0 0 0" />
+        <geometry>
+            <box size="0.001 0.001 0.001" />
+        </geometry>
+    </visual>
+  </link>
+  <!--Base link-->
+  <link name="base_link">
+    <xacro:box_inertia m="10" w="${base_len}" h="${base_width}" d="0.01"/>
+    <visual>
+      <geometry>
+        <box size="${base_len} ${base_width} 0.01"/>
+      </geometry>
+      <material name="black"/>
+    </visual>
+    <collision>
+      <geometry>
+        <box size="${base_len} ${base_width} 0.01"/>
+      </geometry>
+    </collision>
+  </link>
+  <!--base_link to base_footprint Joint-->
+  <joint name="base_link_joint" type="fixed">
+    <origin xyz="0 0 ${wheel_radius + 0.005}" rpy="0 0 0" />
+    <parent link="base_footprint"/>
+    <child link="base_link" />
+  </joint>
+  <!--Wheel link & joint macro-->
+  <xacro:macro name="wheel" params="prefix reflect">
+    <link name="${prefix}_wheel">
+      <visual>
+        <origin xyz="0 0 0" rpy="${pi/2} 0 0"/>
+        <geometry>
+          <cylinder radius="${wheel_radius}" length="0.005"/>
+        </geometry>
+        <material name="red"/>
+      </visual>
+      <collision>
+        <origin xyz="0 0 0" rpy="${pi/2} 0 0"/>
+        <geometry>
+          <cylinder radius="${wheel_radius}" length="0.005"/>
+        </geometry>
+      </collision>
+      <xacro:cylinder_inertia m="10" r="${wheel_radius}" h="0.005"/>
+    </link>
+    <joint name="${prefix}_wheel_joint" type="continuous">
+      <axis xyz="0 1 0" rpy="0 0 0" />
+      <parent link="base_link"/>
+      <child link="${prefix}_wheel"/>
+      <origin xyz="${wheel_joint_offset} ${((base_width/2)+base_wheel_gap)*reflect} -0.005" rpy="0 0 0"/>
+    </joint>
+  </xacro:macro>
+  <!--Create Left & Right Wheel links/joints-->
+  <xacro:wheel prefix="left" reflect="1"/>
+  <xacro:wheel prefix="right" reflect="-1"/>
+  <!--Caster Wheel Link-->
+  <link name="caster_wheel">
+    <visual>
+      <origin xyz="0 0 0" rpy="0 0 0"/>
+      <geometry>
+        <sphere radius="${caster_wheel_radius}"/>
+      </geometry>
+      <material name="blue"/>
+    </visual>
+    <collision>
+      <origin xyz="0 0 0" rpy="0 0 0"/>
+      <geometry>
+        <sphere radius="${caster_wheel_radius}"/>
+      </geometry>
+    </collision>
+    <xacro:sphere_inertia m="10" r="${caster_wheel_radius}"/>
+  </link>
+  <!--Caster Wheel Joint-->
+  <joint name="caster_wheel_joint" type="continuous">
+    <axis xyz="0 1 0" rpy="0 0 0" />
+    <parent link="base_link"/>
+    <child link="caster_wheel"/>
+    <origin xyz="${caster_wheel_joint_offset} 0 -${caster_wheel_radius+0.005}" rpy="0 0 0"/>
+  </joint>
+  <xacro:property name="laser_size_x" value="0.03"/>
+  <xacro:property name="laser_size_y" value="0.03"/>
+  <xacro:property name="laser_size_z" value="0.04"/>
+  <xacro:property name="laser_origin_x" value="0.065"/>
+  <xacro:property name="laser_origin_y" value="0"/>
+  <xacro:property name="laser_origin_z" value="0.035"/>
+  <link name="sensor_laser">
+    <visual>
+      <geometry>
+        <box size="${laser_size_x} ${laser_size_y} ${laser_size_z}"/>
+      </geometry>
+      <material name="blue"/>
+    </visual>
+    <!--visual>
+      <geometry>
+        <mesh filename="package://kbot_description/meshes/hokuyo.dae"/>
+      </geometry>
+    </visual-->
+    <collision>
+      <geometry>
+        <box size="${laser_size_x} ${laser_size_y} ${laser_size_z}"/>
+      </geometry>
+    </collision>
+    <xacro:box_inertia m="0.2" w="${laser_size_x}" h="${laser_size_y}" d="${laser_size_z}"/>
+  </link>
+  <joint name="sensor_laser_joint" type="fixed">
+    <origin xyz="${laser_origin_x} ${laser_origin_y} ${laser_origin_z}" rpy="0 0 0" />
+    <parent link="base_link"/>
+    <child link="sensor_laser" />
+  </joint>
+  <xacro:include filename="$(find robot_description)/urdf/ubot_gazebo_plugins.xacro"/>
 </robot>

Commit message: web interface

File: src/robot_description/urdf/ubot.xacro (robot description, xacro)
@@ -1,8 +1,8 @@
 <?xml version="1.0"?>
 <robot xmlns:xacro="http://www.ros.org/wiki/xacro" name="ubot">
-  <xacro:property name="base_width" value="0.16"/>
-  <xacro:property name="base_len" value="0.16"/>
-  <xacro:property name="wheel_radius" value="0.035"/>
-  <xacro:property name="base_wheel_gap" value="0.007"/>
+  <xacro:property name="base_width" value="0.25"/>
+  <xacro:property name="base_len" value="0.29"/>
+  <xacro:property name="wheel_radius" value="0.032"/>
+  <xacro:property name="base_wheel_gap" value="0.008"/>
   <xacro:property name="wheel_separation" value="0.15"/>
   <xacro:property name="wheel_joint_offset" value="0.02"/>

File: src/robot_description/urdf/ubot_gazebo_plugins.xacro (robot description, xacro)
@@ -34,5 +34,5 @@
         <range>
           <min>0.10</min>
-          <max>30.0</max>
+          <max>3.0</max>
           <resolution>0.01</resolution>
         </range>
